Commit message: removing materials

File: urdfs/leg/leg.gazebo.xacro (robot description, xacro)
@@ -90,5 +90,4 @@
 				</plugin>
 			</sensor>
-			<material>Gazebo/Black</material>
 		</gazebo>
 	</xacro:macro>

File: urdfs/leg/leg.urdf.xacro (robot description, xacro)
@@ -110,5 +110,4 @@
 					<mesh filename="package://hyq_description/meshes/leg/lowerleg.dae" scale="1 1 1"/>
 				</geometry>
-				<material name="white"/>
 			</visual>
 			<collision>
@@ -131,6 +130,5 @@
 					<sphere radius="0.02175" />
 				</geometry>
-				<material name="black" />
-			</visual>
+		</visual>
 		</link>
 		<!-- Extensions -->
