Commit message: added support for new gazebo 11

File: robots/hyq.urdf.xacro (robot description, xacro)
@@ -2,4 +2,5 @@
 <robot name="hyq" xmlns:xacro="http://ros.org/wiki/xacro">
 	<xacro:arg name="task_period" default="0.004"/>
+        <xacro:arg name="new_gazebo_version" default="false"/>
 	<!-- This argument allows us to load joint sensors that measure the internal wrenches -->
 	<xacro:arg name="load_force_sensors" default="false"/>
@@ -24,5 +25,5 @@
 	<!-- body -->
 	<!-- trunk -->
-	<xacro:hyq_trunk name="base">
+        <xacro:hyq_trunk name="base" new_gazebo_version="$(arg new_gazebo_version)">
 		<!--origin xyz="-0.443 -0.191 -0.276" rpy="0 0 0"/-->
 	</xacro:hyq_trunk>

File: urdfs/trunk/trunk.urdf.xacro (robot description, xacro)
@@ -5,16 +5,20 @@
 	<!-- ================================ Trunk ================================ -->
 	<!-- The xacro macro xacro:hyq_base contains: base and trunk -->
-	<xacro:macro name="hyq_trunk" params="name">
-		  <!-- Floating-base Joint -->
-                <link name="world"/>
-                <joint name="floating_base_joint" type="floating">
-                  <origin rpy="0 0 0" xyz="0 0 0"/>
-                  <parent link="world"/>
-                  <child link="base_link"/>
-                </joint>
+        <xacro:macro name="hyq_trunk" params="name new_gazebo_version">
+                <!-- BASE LINK -->
+                <!-- floating type is supported in older versions of Gazebo. In new Gazebo if a link has no parent, it is supposed to be attached to a floating joint -->
+                <xacro:unless value="$(arg new_gazebo_version)">
+                    <!-- Floating-base Joint -->
+                    <link name="world"/>
+                    <joint name="floating_base_joint" type="floating" >
+                        <origin rpy="0 0 0" xyz="0 0 0"/>
+                        <parent link="world"/>
+                        <child link="base_link"/>
+                    </joint>
+                </xacro:unless>
                 <joint name="floating_base" type="fixed">
-                  <origin rpy="0 0 0" xyz="0 0 0"/>
-                  <parent link="base_link"/>
-                  <child link="trunk"/>
+                    <origin rpy="0 0 0" xyz="0 0 0"/>
+                    <parent link="base_link"/>
+                    <child link="trunk"/>
                 </joint>
 		<!-- Links -->

Commit message: finally fixing the hack of new_gazebo_version to set root joint for pinocchio as per robot_control commit fccb58b1fb819f6c18701ba5d1a20bd6d21af330

File: robots/hyq.urdf.xacro (robot description, xacro)
@@ -2,5 +2,4 @@
 <robot name="hyq" xmlns:xacro="http://ros.org/wiki/xacro">
 	<xacro:arg name="task_period" default="0.004"/>
-        <xacro:arg name="new_gazebo_version" default="false"/>
 	<!-- This argument allows us to load joint sensors that measure the internal wrenches -->
 	<xacro:arg name="load_force_sensors" default="false"/>
@@ -25,5 +24,5 @@
 	<!-- body -->
 	<!-- trunk -->
-        <xacro:hyq_trunk name="base" new_gazebo_version="$(arg new_gazebo_version)">
+        <xacro:hyq_trunk name="base">
 		<!--origin xyz="-0.443 -0.191 -0.276" rpy="0 0 0"/-->
 	</xacro:hyq_trunk>

File: urdfs/trunk/trunk.urdf.xacro (robot description, xacro)
@@ -5,16 +5,5 @@
 	<!-- ================================ Trunk ================================ -->
 	<!-- The xacro macro xacro:hyq_base contains: base and trunk -->
-        <xacro:macro name="hyq_trunk" params="name new_gazebo_version">
-                <!-- BASE LINK -->
-                <!-- floating type is supported in older versions of Gazebo. In new Gazebo if a link has no parent, it is supposed to be attached to a floating joint -->
-                <xacro:unless value="$(arg new_gazebo_version)">
-                    <!-- Floating-base Joint -->
-                    <link name="world"/>
-                    <joint name="floating_base_joint" type="floating" >
-                        <origin rpy="0 0 0" xyz="0 0 0"/>
-                        <parent link="world"/>
-                        <child link="base_link"/>
-                    </joint>
-                </xacro:unless>
+        <xacro:macro name="hyq_trunk" params="name">
                 <joint name="floating_base" type="fixed">
                     <origin rpy="0 0 0" xyz="0 0 0"/>
